File: Kicad/Stepper Module.kicad_pcb (KiCad board)
At the start: 4 copper layers, 97.8 x 99.6 mm, 169 parts, among them J1 2.0_16P, J11 OLED, J12 Conn_02x05_Odd_Even, J13 Conn_02x05_Odd_Even, J2 esp12F-CHARG, J3 BAT, J4 FRC Conn, J5 ESP12F_PROG, J6 PICO Debug, J7 ESP32_PROG, J8 OLED, SW1 UP, SW10 esp32nowAddress, SW11 esp12fnowAddress, SW12 12E_NEXT, SW13 12E_PRV, SW14 12E_Enter, SW15 Reset, SW16 BOOTSEL, SW17 Reset, SW2 PRV, SW3 NEXT, SW4 DOWN, SW5 SELECT, SW6 EXIT, SW7 NEXT_0, SW8 PRV_0, SW9 SELECT_0, T40 ADC3, T41 ADC2, T42 VREG, U1 LM2596S-ADJ, U2 TMC2209-LA-T, U5 ESP-12F, U7 RP2040, U8 W25Q32JVSS, Y1 FA-20H-12-10

Commit message: PCB design Changes
Parts:
- added C30: C_Polarized_Small, Capacitor_Tantalum_SMD:CP_EIA-3528-21_Kemet-B, B.Cu at (162.9, 94.7)
- added C31: C_Polarized_Small, Capacitor_Tantalum_SMD:CP_EIA-3528-21_Kemet-B, B.Cu at (150.8, 94.7)
- added D11: SS14, Diode_SMD:D_SMA, B.Cu at (157.6, 87.0)
- added U9: AMS1117-3.3, Package_TO_SOT_SMD:SOT-223-3_TabPin2, B.Cu at (156.9, 93.6)
- R10: value R_US -> Rsens/9-12v
- moved TP8 0.06 mm to (179.2, 96.0)
Connections:
- net E12F_FLASH renamed E12F_CS
- net ESP32_FL_EN renamed ESP32_CS
- C10 pad 2: Vdrive -> +5VD
- C12 pad 2: Vlogic -> Vdrive
- C6 pad 2: Vlogic -> Vdrive
- C7 pad 1: Vlogic -> Vdrive
- D4 pad 2: Vlogic -> Vdrive
- J4 pad 10: Vmotor -> Vdrive
- J4 pad 7: Vlogic -> Vmotor
- L1 pad 2: Vlogic -> Vdrive
- R1 pad 1: Vdrive -> +5VD
- R10 pad 1: Vlogic -> Vdrive
- R2 pad 2: Vdrive -> +5VD
- TP7 pad 1: Vdrive -> +5VD
- U2 pad 8: Vdrive -> +5VD
Routing:
- net Vdrive: track 11.9 -> 53.4 mm, vias 0 -> 14
- net (no net): track 19.3 -> 0.00 mm
- net Net-(D11-A): track 0.00 -> 17.2 mm
- net Vlogic: track 109.2 -> 94.3 mm, vias 25 -> 23
- net +5VD: track 0.00 -> 11.9 mm
- net GND: track 611.4 -> 604.6 mm, vias 47 -> 49
- net BMS_GND: track 99.9 -> 105.2 mm
- net ESP32_CS: track 30.5 -> 34.6 mm
- net Vmotor: track 78.6 -> 81.3 mm
- net /SELECT: track 44.8 -> 43.0 mm
- net ESP32_0TX: track 6.62 -> 8.37 mm
- net ESP32_EN: track 10.2 -> 11.6 mm
- net OB2: track 31.9 -> 31.0 mm
- net ESP32_0RX: track 9.00 -> 9.85 mm
- net OA1: track 38.8 -> 39.6 mm
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- added copper zone on B.Cu, net Vdrive
- added copper zone on F.Cu, net Vdrive
- added copper zone on In2.Cu, net Vdrive
- removed copper zone on F.Cu, net Vlogic

Commit message: final send
Parts:
- removed JP3: SolderJumper_2_Open, Jumper:SolderJumper-2_P1.3mm_Open_TrianglePad1.0x1.5mm
Connections:
- D2 pad 1: 5Vout -> Vdrive
- H1 pad : (no net) -> GND
- H2 pad : (no net) -> GND
- H3 pad : (no net) -> GND
- H4 pad : (no net) -> GND
- H5 pad : (no net) -> GND
- H6 pad : (no net) -> GND
- H7 pad : (no net) -> GND
- H8 pad : (no net) -> GND
- TP6 pad 1: 5Vout -> Vdrive
Routing:
- net GND: track 604.6 -> 805.5 mm
- net Vmotor: track 81.3 -> 56.7 mm
- net Vdrive: track 53.4 -> 62.7 mm
- net 5Vout: track 7.39 -> 0.00 mm
- net OA1: track 39.6 -> 38.4 mm
- net HALL: track 97.9 -> 98.6 mm

Commit message: First update PCB V1
Parts:
- removed R32: 10KR, Resistor_SMD:R_0805_2012Metric
Connections:
- H1 pad : GND -> (no net)
- H2 pad : GND -> (no net)
- H3 pad : GND -> (no net)
- H4 pad : GND -> (no net)
- H5 pad : GND -> (no net)
- H6 pad : GND -> (no net)
- H7 pad : GND -> (no net)
- H8 pad : GND -> (no net)
Routing:
- net /LED_esp12: track 11.5 -> 8.65 mm
- net BMS_GND: track 105.2 -> 102.8 mm
- net Vmotor: track 56.7 -> 54.9 mm
- added copper zone on F.Cu, net Vlogic
