File: Kicad/Stepper Module.kicad_sch (KiCad schematic)
At the start: 169 parts, among them J1 2.0_16P, J11 OLED, J12 Conn_02x05_Odd_Even, J13 Conn_02x05_Odd_Even, J2 esp12F-CHARG, J3 BAT, J4 FRC Conn, J5 ESP12F_PROG, J6 PICO Debug, J7 ESP32_PROG, J8 OLED, SW1 UP, SW10 esp32nowAddress, SW11 esp12fnowAddress, SW12 12E_NEXT, SW13 12E_PRV, SW14 12E_Enter, SW15 Reset, SW16 BOOTSEL, SW17 Reset, SW2 PRV, SW3 NEXT, SW4 DOWN, SW5 SELECT, SW6 EXIT, SW7 NEXT_0, SW8 PRV_0, SW9 SELECT_0, T40 ADC3, T41 ADC2, T42 VREG, U1 LM2596S-ADJ, U2 TMC2209-LA-T, U5 ESP-12F, U6 ESP32-WROOM-32D, U7 RP2040, U8 W25Q32JVSS, Y1 FA-20H-12-10

Commit message: PCB design Changes
Parts:
- added C30, C31: C_Polarized_Small, Capacitor_Tantalum_SMD:CP_EIA-3528-21_Kemet-B, symbol Device:C_Polarized_Small
- added D11: SS14, Diode_SMD:D_SMA, symbol Device:D_Schottky
- added U9: AMS1117-3.3, Package_TO_SOT_SMD:SOT-223-3_TabPin2, symbol Regulator_Linear:AMS1117-3.3
- R10: value R_US -> Rsens/9-12v
Connections:
- net +12V: now also J4.7 (Pin_7); no longer J4.10 (Pin_10)
- net +3V3: now also D11.1 (K); no longer C12.2, C6.2, C7.1, D4.2 (A), J4.7 (Pin_7), L1.2, R10.1
- net GND: now also C30.2, C31.2, U9.1 (GND)
- net Vdrive: now also C12.2, C6.2, C7.1, D4.2 (A), J4.10 (Pin_10), L1.2, R10.1, C30.1, U9.3 (VI); no longer C10.2, R1.1, R2.2, TP7.1, U2.8 (5VOUT)
- net E12F_FLASH renamed E12F_CS
- net ESP32_FL_EN renamed ESP32_CS
- new net: C31.1, D11.2 (A), U9.2 (VO)
- new net +5VD: C10.2, R1.1, R2.2, TP7.1, U2.8 (5VOUT)
Other:
- note added: "OLED_I2C_PRI"
- note added: "OLED_I2C_SEC"
- note added: "Wired Keypad-Oled Extention Connectors"
- note added: "Wireless controller charging & PSU"
- note removed: "OLED_I2C"
- note removed: "OLED_I2C_Out"
- note removed: "Wireless comtrpller charging & PSU"
- moved on the sheet: C13, C14, C6, D7, D8, D9, H1, H2, H3, H4, H5, H6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

Commit message: final send
Parts:
- removed JP3: SolderJumper_2_Open, Jumper:SolderJumper-2_P1.3mm_Open_TrianglePad1.0x1.5mm, symbol Jumper:SolderJumper_2_Open
Connections:
- net Vdrive is gone; now on net +5V: C12.2, C30.1, C6.2, C7.1, D4.2 (A), J4.10 (Pin_10), L1.2, R10.1, U9.3 (VI)
- no-connect marks 20 -> 21
Other:
- note added: "9-12v OUT for Sensors & 1117-3v3"

Commit message: First update PCB V1
Parts:
- removed R32: 10KR, Resistor_SMD:R_0805_2012Metric, symbol Device:R
- added D?: LED, symbol Device:LED
- added R?: 10KR, Resistor_SMD:R_0805_2012Metric, symbol Device:R
- added R?: Rpri, symbol Device:R
- added R?: R 1k, symbol Device:R
- added R?: Rsec, symbol Device:R
- added U?: PC817, Package_DIP:DIP-4_W7.62mm, symbol Isolator:PC817
- added U?: Hall Sensor, Package_TO_SOT_SMD:SOT-23, symbol Sensor_Magnetic:SM351LT
Connections:
- net +3V3: now also R?.2, R?.2
- net 12E_Enter: no longer U5.4 (GPIO16)
- net 12FADD00: no longer U5.16 (GPIO15)
- net 12FADD01: no longer U5.7 (GPIO13)
- net GND: now also U?.3 (GND)
- net GND2: now also R?.2
- new net: R?.1, U5.16 (GPIO15)
- new net: R?.2, U?.1
- new net: U?.2, U?.2 (OUTPUT)
- new net: D?.2 (A), R?.1
- new net -12V: R?.1, U?.1 (VCC)
- new net Earth: U?.3
- new net Signal Output: D?.1 (K), R?.1, U?.4
